Commit message: Adjusted Position od Laserscanner
Co-authored-by: Copilot <copilot@github.com>

File: src/mensabot_description/urdf/mensabot.urdf.xacro (robot description, xacro)
@@ -386,5 +386,5 @@
   <!--FRONT LASER SCANNER  -->
   <joint type="fixed" name="scan_front_joint">
-    <origin xyz="0.4 0.33 0.1" rpy="0 0 0.7854"/>     <!--origin xyz="0.3775 0.314 0.1" rpy="0 0 0"/-->
+    <origin xyz="0.3875 0.28 0.1" rpy="0 0 0.8054"/>     <!--origin xyz="0.3775 0.314 0.1" rpy="0 0 0"/-->
     <child link="scan_front_link"/>
     <parent link="center_link"/>
@@ -408,5 +408,5 @@
   <!--REAR LASER SCANNER  -->
   <joint type="fixed" name="scan_rear_joint">
-    <origin xyz="-0.4 -0.33 0.1" rpy="0 0 3.927"/>
+    <origin xyz="-0.3875 -0.28 0.1" rpy="0 0 3.927"/>
     <child link="scan_rear_link"/>
     <parent link="center_link"/>
