Commit message: Added launch for Safetyscanners, updated URDF for LIDAR Position

File: src/mensabot_description/urdf/mensabot.urdf.xacro (robot description, xacro)
@@ -386,5 +386,5 @@
   <!--FRONT LASER SCANNER  -->
   <joint type="fixed" name="scan_front_joint">
-    <origin xyz="0.4 0.33 0.1" rpy="0 0 0"/>     <!--origin xyz="0.3775 0.314 0.1" rpy="0 0 0"/-->
+    <origin xyz="0.4 0.33 0.1" rpy="0 0 0.7854"/>     <!--origin xyz="0.3775 0.314 0.1" rpy="0 0 0"/-->
     <child link="scan_front_link"/>
     <parent link="center_link"/>
@@ -408,5 +408,5 @@
   <!--REAR LASER SCANNER  -->
   <joint type="fixed" name="scan_rear_joint">
-    <origin xyz="-0.4 -0.33 0.1" rpy="0 0 ${pi}"/>
+    <origin xyz="-0.4 -0.33 0.1" rpy="0 0 3.927"/>
     <child link="scan_rear_link"/>
     <parent link="center_link"/>

Commit message: Updated URDF for new Position of Lidars

File: src/mensabot_description/urdf/mensabot.urdf.xacro (robot description, xacro)
@@ -34,5 +34,5 @@
     </collision>
     <collision name='left_caster_collision'>
-      <origin xyz="-0.45 0.2 -0.0475" rpy=" 0 0 0"/>
+      <origin xyz="-0.4 0.2 -0.0475" rpy=" 0 0 0"/>
       <geometry>
         <sphere radius="0.0625"/>
@@ -40,5 +40,5 @@
     </collision>
     <visual name='left_caster_visual'>
-      <origin xyz="-0.45 0.2 -0.0475 " rpy=" 0 0 0"/>
+      <origin xyz="-0.4 0.2 -0.0475 " rpy=" 0 0 0"/>
       <geometry>
         <sphere radius="0.0625"/>
@@ -47,5 +47,5 @@
     </visual>
     <collision name='right_caster_collision'>
-      <origin xyz="-0.45 -0.2 -0.0475" rpy=" 0 0 0"/>
+      <origin xyz="-0.4 -0.2 -0.0475" rpy=" 0 0 0"/>
       <geometry>
         <sphere radius="0.0625"/>
@@ -53,5 +53,5 @@
     </collision>
     <visual name='right_caster_visual'>
-      <origin xyz="-0.45 -0.2 -0.0475" rpy=" 0 0 0"/>
+      <origin xyz="-0.4 -0.2 -0.0475" rpy=" 0 0 0"/>
       <geometry>
         <sphere radius="0.0625"/>
@@ -65,5 +65,5 @@
   <!--CENTER LINK-->
   <joint name="center_joint" type="fixed">
-    <origin xyz="-0.2 0 0" rpy="0 0 0" />
+    <origin xyz="-0.15 0 0" rpy="0 0 0" />
     <parent link="base_link"/>
     <child link="center_link" />
@@ -185,5 +185,5 @@
   <!-- Vertical Rods -->
   <joint name="front_right1_joint" type="fixed">
-    <origin xyz="0.355 0.2015 0.1475" rpy="0 ${pi/2} 0" />
+    <origin xyz="0.31 0.2015 0.1475" rpy="0 ${pi/2} 0" />
     <parent link="center_link"/>
     <child link="front_right1_link" />
@@ -198,5 +198,5 @@
   </link>
   <joint name="front_left1_joint" type="fixed">
-    <origin xyz="0.355 -0.2015 0.1475" rpy="0 ${pi/2} 0" />
+    <origin xyz="0.31 -0.2015 0.1475" rpy="0 ${pi/2} 0" />
     <parent link="center_link"/>
     <child link="front_left1_link" />
@@ -210,76 +210,50 @@
     </visual>
   </link>
-  <joint name="front_right2_joint" type="fixed">
-    <origin xyz="0.265 0.2915 0.1475" rpy="0 ${pi/2} 0" />
-    <parent link="center_link"/>
-    <child link="front_right2_link" />
-  </joint>
-  <link name="front_right2_link">
-    <visual name='front_right2_visual'>
-       <geometry>
-         <box size="0.25 0.045 0.045"/>
-       </geometry>
-       <material name="grey"/>
-    </visual>
-  </link>
-  <joint name="front_left2_joint" type="fixed">
-    <origin xyz="0.265 -0.2915 0.1475" rpy="0 ${pi/2} 0" />
-    <parent link="center_link"/>
-    <child link="front_left2_link" />
-  </joint>
-  <link name="front_left2_link">
-    <visual name='front_left2_visual'>
-       <geometry>
-         <box size="0.25 0.045 0.045"/>
-       </geometry>
-       <material name="grey"/>
-    </visual>
-  </link>
-  <joint name="back_left1_joint" type="fixed">
-    <origin xyz="-0.355 -0.2015 0.1475" rpy="0 ${pi/2} 0" />
-    <parent link="center_link"/>
-    <child link="back_left1_link" />
-  </joint>
-  <link name="back_left1_link">
-    <visual name='back_left1_visual'>
-       <geometry>
-         <box size="0.25 0.045 0.045"/>
-       </geometry>
-       <material name="grey"/>
-    </visual>
-  </link>
-  <joint name="back_right1_joint" type="fixed">
-    <origin xyz="-0.355 0.2015 0.1475" rpy="0 ${pi/2} 0" />
-    <parent link="center_link"/>
-    <child link="back_right1_link" />
-  </joint>
-  <link name="back_right1_link">
-    <visual name='back_right1_visual'>
-       <geometry>
-         <box size="0.25 0.045 0.045"/>
-       </geometry>
-       <material name="grey"/>
-    </visual>
-  </link>
-  <joint name="back_left2_joint" type="fixed">
-    <origin xyz="-0.265 -0.2915 0.1475" rpy="0 ${pi/2} 0" />
-    <parent link="center_link"/>
-    <child link="back_left2_link" />
-  </joint>
-  <link name="back_left2_link">
-    <visual name='back_left2_visual'>
-       <geometry>
-         <box size="0.25 0.045 0.045"/>
-       </geometry>
-       <material name="grey"/>
-    </visual>
-  </link>
-  <joint name="back_right2_joint" type="fixed">
-    <origin xyz="-0.265 0.2915 0.1475" rpy="0 ${pi/2} 0" />
-    <parent link="center_link"/>
-    <child link="back_right2_link" />
-  </joint>
-  <link name="back_right2_link">
-    <visual name='back_right2_visual'>
+  <joint name="right_joint" type="fixed">
+    <origin xyz="0 0.2465 0.1475" rpy="0 ${pi/2} 0" />
+    <parent link="center_link"/>
+    <child link="right_link" />
+  </joint>
+  <link name="right_link">
+    <visual name='right_visual'>
+       <geometry>
+         <box size="0.25 0.045 0.045"/>
+       </geometry>
+       <material name="grey"/>
+    </visual>
+  </link>
+  <joint name="_left_joint" type="fixed">
+    <origin xyz="0 -0.2465 0.1475" rpy="0 ${pi/2} 0" />
+    <parent link="center_link"/>
+    <child link="left_link" />
+  </joint>
+  <link name="left_link">
+    <visual name='left_visual'>
+       <geometry>
+         <box size="0.25 0.045 0.045"/>
+       </geometry>
+       <material name="grey"/>
+    </visual>
+  </link>
+  <joint name="back_left_joint" type="fixed">
+    <origin xyz="-0.315 -0.2015 0.1475" rpy="0 ${pi/2} 0" />
+    <parent link="center_link"/>
+    <child link="back_left_link" />
+  </joint>
+  <link name="back_left_link">
+    <visual name='back_left_visual'>
+       <geometry>
+         <box size="0.25 0.045 0.045"/>
+       </geometry>
+       <material name="grey"/>
+    </visual>
+  </link>
+  <joint name="back_right_joint" type="fixed">
+    <origin xyz="-0.315 0.2015 0.1475" rpy="0 ${pi/2} 0" />
+    <parent link="center_link"/>
+    <child link="back_right_link" />
+  </joint>
+  <link name="back_right_link">
+    <visual name='back_right_visual'>
        <geometry>
          <box size="0.25 0.045 0.045"/>

Commit message: Update URDF to Real Robot Dimnesions and Lidar Positions

File: src/mensabot_description/urdf/mensabot.urdf.xacro (robot description, xacro)
@@ -28,5 +28,5 @@
   <link name='base_link'>
     <collision name="base_collision">
-      <origin xyz="-0.2 0 0.15" rpy="0 0 0"/>       <!-- Collision geometry -->
+      <origin xyz="-0.1775 0 0.15" rpy="0 0 0"/>       <!-- Collision geometry -->
       <geometry>
         <box size="0.7 0.55 0.01"/>
@@ -34,5 +34,5 @@
     </collision>
     <collision name='left_caster_collision'>
-      <origin xyz="-0.4 0.2 -0.0475" rpy=" 0 0 0"/>
+      <origin xyz="-0.445 0.2 -0.0475" rpy=" 0 0 0"/>
       <geometry>
         <sphere radius="0.0625"/>
@@ -40,5 +40,5 @@
     </collision>
     <visual name='left_caster_visual'>
-      <origin xyz="-0.4 0.2 -0.0475 " rpy=" 0 0 0"/>
+      <origin xyz="-0.445 0.2 -0.0475 " rpy=" 0 0 0"/>
       <geometry>
         <sphere radius="0.0625"/>
@@ -47,5 +47,5 @@
     </visual>
     <collision name='right_caster_collision'>
-      <origin xyz="-0.4 -0.2 -0.0475" rpy=" 0 0 0"/>
+      <origin xyz="-0.445 -0.2 -0.0475" rpy=" 0 0 0"/>
       <geometry>
         <sphere radius="0.0625"/>
@@ -53,5 +53,5 @@
     </collision>
     <visual name='right_caster_visual'>
-      <origin xyz="-0.4 -0.2 -0.0475" rpy=" 0 0 0"/>
+      <origin xyz="-0.445 -0.2 -0.0475" rpy=" 0 0 0"/>
       <geometry>
         <sphere radius="0.0625"/>
@@ -65,5 +65,5 @@
   <!--CENTER LINK-->
   <joint name="center_joint" type="fixed">
-    <origin xyz="-0.15 0 0" rpy="0 0 0" />
+    <origin xyz="-0.1775 0 0" rpy="0 0 0" />
     <parent link="base_link"/>
     <child link="center_link" />
@@ -79,5 +79,5 @@
 <!-- Bottom Layer -->
   <joint name="bottom_front_rod_joint" type="fixed">
-    <origin xyz="0.355 0 0" rpy="0 0 ${pi/2}" />
+    <origin xyz="0.4 0 0" rpy="0 0 ${pi/2}" />
     <parent link="center_link"/>
     <child link="bottom_front_rod_link" />
@@ -86,5 +86,5 @@
     <visual name='bottom_front_rod_visual'>
        <geometry>
-         <box size="0.538 0.045 0.045"/>
+         <box size="0.520 0.045 0.045"/>
        </geometry>
        <material name="grey"/>
@@ -92,5 +92,5 @@
   </link>
   <joint name="bottom_rear_rod_joint" type="fixed">
-    <origin xyz="-0.355 0 0" rpy="0 0 ${pi/2}" />
+    <origin xyz="-0.4 0 0" rpy="0 0 ${pi/2}" />
     <parent link="center_link"/>
     <child link="bottom_rear_rod_link" />
@@ -99,5 +99,5 @@
     <visual name='bottom_rear_rod_visual'>
        <geometry>
-         <box size="0.538 0.045 0.045"/>
+         <box size="0.520 0.045 0.045"/>
        </geometry>
        <material name="grey"/>
@@ -105,5 +105,5 @@
   </link>
   <joint name="bottom_left_rod_joint" type="fixed">
-    <origin xyz="0.0 0.2915 0" rpy="0 0 0" />
+    <origin xyz="0.0 0.2825 0" rpy="0 0 0" />
     <parent link="center_link"/>
     <child link="bottom_left_rod_link" />
@@ -118,5 +118,5 @@
   </link>
   <joint name="bottom_right_rod_joint" type="fixed">
-    <origin xyz="0.0 -0.2915 0" rpy="0 0 0" />
+    <origin xyz="0.0 -0.2825 0" rpy="0 0 0" />
     <parent link="center_link"/>
     <child link="bottom_right_rod_link" />
@@ -139,5 +139,5 @@
     <visual name='top_front_rod_visual'>
        <geometry>
-         <box size="0.538 0.045 0.045"/>
+         <box size="0.446 0.045 0.045"/>
        </geometry>
        <material name="grey"/>
@@ -152,5 +152,5 @@
     <visual name='top_rear_rod_visual'>
        <geometry>
-         <box size="0.538 0.045 0.045"/>
+         <box size="0.446 0.045 0.045"/>
        </geometry>
        <material name="grey"/>
@@ -158,5 +158,5 @@
   </link>
   <joint name="top_left_rod_joint" type="fixed">
-    <origin xyz="0.0 0.2915 0.295" rpy="0 0 0" />
+    <origin xyz="0.0 0.2375 0.295" rpy="0 0 0" />
     <parent link="center_link"/>
     <child link="top_left_rod_link" />
@@ -171,5 +171,5 @@
   </link>
   <joint name="top_right_rod_joint" type="fixed">
-    <origin xyz="0.0 -0.2915 0.295" rpy="0 0 0" />
+    <origin xyz="0.0 -0.2375 0.295" rpy="0 0 0" />
     <parent link="center_link"/>
     <child link="top_right_rod_link" />
@@ -185,5 +185,5 @@
   <!-- Vertical Rods -->
   <joint name="front_right1_joint" type="fixed">
-    <origin xyz="0.31 0.2015 0.1475" rpy="0 ${pi/2} 0" />
+    <origin xyz="0.355 0.2015 0.1475" rpy="0 ${pi/2} 0" />
     <parent link="center_link"/>
     <child link="front_right1_link" />
@@ -198,5 +198,5 @@
   </link>
   <joint name="front_left1_joint" type="fixed">
-    <origin xyz="0.31 -0.2015 0.1475" rpy="0 ${pi/2} 0" />
+    <origin xyz="0.355 -0.2015 0.1475" rpy="0 ${pi/2} 0" />
     <parent link="center_link"/>
     <child link="front_left1_link" />
@@ -211,5 +211,5 @@
   </link>
   <joint name="right_joint" type="fixed">
-    <origin xyz="0 0.2465 0.1475" rpy="0 ${pi/2} 0" />
+    <origin xyz="0 0.2375 0.1475" rpy="0 ${pi/2} 0" />
     <parent link="center_link"/>
     <child link="right_link" />
@@ -223,6 +223,6 @@
     </visual>
   </link>
-  <joint name="_left_joint" type="fixed">
-    <origin xyz="0 -0.2465 0.1475" rpy="0 ${pi/2} 0" />
+  <joint name="left_joint" type="fixed">
+    <origin xyz="0 -0.2375 0.1475" rpy="0 ${pi/2} 0" />
     <parent link="center_link"/>
     <child link="left_link" />
@@ -237,5 +237,5 @@
   </link>
   <joint name="back_left_joint" type="fixed">
-    <origin xyz="-0.315 -0.2015 0.1475" rpy="0 ${pi/2} 0" />
+    <origin xyz="-0.355 -0.2015 0.1475" rpy="0 ${pi/2} 0" />
     <parent link="center_link"/>
     <child link="back_left_link" />
@@ -250,5 +250,5 @@
   </link>
   <joint name="back_right_joint" type="fixed">
-    <origin xyz="-0.315 0.2015 0.1475" rpy="0 ${pi/2} 0" />
+    <origin xyz="-0.355 0.2015 0.1475" rpy="0 ${pi/2} 0" />
     <parent link="center_link"/>
     <child link="back_right_link" />
@@ -343,5 +343,5 @@
   </gazebo>
   <joint name="imu_joint" type="fixed">
-    <origin xyz="0.0 0 0.05" rpy="0 0 0" />
+    <origin xyz="0.0 0.2375 0.05" rpy="0 0 0" />
     <parent link="base_link"/>
     <child link="imu_link" />
@@ -360,5 +360,5 @@
   <!--FRONT LASER SCANNER  -->
   <joint type="fixed" name="scan_front_joint">
-    <origin xyz="0.3875 0.28 0.1" rpy="0 0 0.8054"/>     <!--origin xyz="0.3775 0.314 0.1" rpy="0 0 0"/-->
+    <origin xyz="0.3875 -0.28 0.08" rpy="0 3.1415 2.3562"/>     <!--Lidar height is 19cm above ground-->
     <child link="scan_front_link"/>
     <parent link="center_link"/>
@@ -382,5 +382,5 @@
   <!--REAR LASER SCANNER  -->
   <joint type="fixed" name="scan_rear_joint">
-    <origin xyz="-0.3875 -0.28 0.1" rpy="0 0 3.927"/>
+    <origin xyz="-0.3875 0.28 0.08" rpy="0 3.1415 -0.7654"/>    <!--Lidar height is 19cm above ground-->
     <child link="scan_rear_link"/>
     <parent link="center_link"/>

Commit message: Updated real Robot values and Topics to Simulation

File: src/mensabot_description/urdf/mensabot.urdf.xacro (robot description, xacro)
@@ -343,5 +343,5 @@
   </gazebo>
   <joint name="imu_joint" type="fixed">
-    <origin xyz="0.0 0.2375 0.05" rpy="0 0 0" />
+    <origin xyz="0.0 0.0 0.25" rpy="0 0 0" />
     <parent link="base_link"/>
     <child link="imu_link" />

Commit message: Updated Position of Lidar to fit scans

File: src/mensabot_description/urdf/mensabot.urdf.xacro (robot description, xacro)
@@ -360,5 +360,5 @@
   <!--FRONT LASER SCANNER  -->
   <joint type="fixed" name="scan_front_joint">
-    <origin xyz="0.3875 -0.28 0.08" rpy="0 3.1415 2.3562"/>     <!--Lidar height is 19cm above ground-->
+    <origin xyz="0.3875 -0.28 0.08" rpy="0 3.1415 2.3562"/>     <!-- <origin xyz="0.3875 -0.28 0.08" rpy="0 3.1415 2.3562"/> Lidar height is 18cm above ground -->
     <child link="scan_front_link"/>
     <parent link="center_link"/>
@@ -382,5 +382,5 @@
   <!--REAR LASER SCANNER  -->
   <joint type="fixed" name="scan_rear_joint">
-    <origin xyz="-0.3875 0.28 0.08" rpy="0 3.1415 -0.7654"/>    <!--Lidar height is 19cm above ground-->
+    <origin xyz="-0.3875 0.28 0.08" rpy="0 3.1415 -0.7854"/>    <!-- <origin xyz="-0.3875 0.28 0.08" rpy="0 3.1415 -0.7654"/> Lidar height is 18cm above ground-->
     <child link="scan_rear_link"/>
     <parent link="center_link"/>
