Commit message: Adjustments to IMU and EKF

File: src/mensabot_description/urdf/mensabot.urdf.xacro (robot description, xacro)
@@ -343,5 +343,5 @@
   </gazebo>
   <joint name="imu_joint" type="fixed">
-    <origin xyz="0.0 0.0 0.25" rpy="0 0 0" />
+  <origin xyz="0.0 -0.01 0.25" rpy="0 0 0" /> <!-- Real Rotation centre of the IMU is not in the centre of the Hardware -->
     <parent link="base_link"/>
     <child link="imu_link" />

Commit message: Finaly removed pld package mensabot_sim entirely

File: src/mensabot_description/urdf/mensabot.urdf.xacro (robot description, xacro)
@@ -343,5 +343,5 @@
   </gazebo>
   <joint name="imu_joint" type="fixed">
-  <origin xyz="0.0 -0.01 0.25" rpy="0 0 0" /> <!-- Real Rotation centre of the IMU is not in the centre of the Hardware -->
+  <origin xyz="0.0 0.0 0.25" rpy="0 0 0" />
     <parent link="base_link"/>
     <child link="imu_link" />
